File: Hardware/Qwiic_BMA456.kicad_pcb (KiCad board)
At the start: 2 copper layers, 25.4 x 25.4 mm, 63 parts, among them J0 LED, J1 Conn_01x04, J2 Qwiic_RA, J3 I²C, J4 Qwiic_RA, J5 Conn_01x06, J6 ADDR, U1 KX134

Commit message: Design Review Changes
Parts:
- removed G1: OSHW_Logo, SparkFun-Aesthetic:Creative_Commons_License
- removed kibuzzard-6A2AF6B9: G***, kibuzzard-6A2AF6B9
- removed kibuzzard-6A2AF6DB: G***, kibuzzard-6A2AF6DB
- removed kibuzzard-6A8485B7: G***, kibuzzard-6A8485B7
- removed kibuzzard-6A848DA7: G***, kibuzzard-6A848DA7
- removed kibuzzard-6A848DB2: G***, kibuzzard-6A848DB2
- removed kibuzzard-6A848DEC: G***, kibuzzard-6A848DEC
- removed kibuzzard-6A848DF0: G***, kibuzzard-6A848DF0
- removed kibuzzard-6A849B08: G***, kibuzzard-6A849B08
- removed kibuzzard-6A849B0E: G***, kibuzzard-6A849B0E
- removed kibuzzard-6A84B32C: G***, kibuzzard-6A84B32C
- added kibuzzard-6A8DBB71: G***, kibuzzard-6A8DBB71, B.Cu at (150.5, 79.4)
- added kibuzzard-6A8DBB79: G***, kibuzzard-6A8DBB79, B.Cu at (150.8, 80.6)
- added kibuzzard-6A8DBBAF: G***, kibuzzard-6A8DBBAF, F.Cu at (147.3, 73.0)
- added kibuzzard-6A8DBBAF: G***, kibuzzard-6A8DBBAF, B.Cu at (147.3, 73.0)
- added kibuzzard-6A8DBBBE: G***, kibuzzard-6A8DBBBE, F.Cu at (149.9, 73.0)
- added kibuzzard-6A8DBBBE: G***, kibuzzard-6A8DBBBE, B.Cu at (149.9, 73.0)
- added kibuzzard-6A8DBBCD: G***, kibuzzard-6A8DBBCD, F.Cu at (152.4, 73.3)
- added kibuzzard-6A8DBBCD: G***, kibuzzard-6A8DBBCD, B.Cu at (152.4, 73.3)
- added kibuzzard-6A8DBBD9: G***, kibuzzard-6A8DBBD9, F.Cu at (154.9, 73.3)
- added kibuzzard-6A8DBBD9: G***, kibuzzard-6A8DBBD9, B.Cu at (154.9, 73.3)
- added kibuzzard-6A8DC94F: G***, kibuzzard-6A8DC94F, B.Cu at (149.4, 82.7)
- added kibuzzard-6A8DC959: G***, kibuzzard-6A8DC959, B.Cu at (147.5, 82.7)
- U1: value KX134 -> BMA456
- moved G*** 13.3 mm to (157.8, 86.4)
- moved kibuzzard-6A848A2E 0.34 mm to (147.8, 88.7)
- moved kibuzzard-6A8489CE 0.34 mm to (145.7, 86.5)
- moved kibuzzard-6A848A36 0.34 mm to (148.2, 85.3)
- turned J6 to 180 degrees
- turned R4 to 180 degrees
Connections:
- J6 pad 1: GND -> Net-(J6-A)
- J6 pad 3: Net-(J6-C) -> 3.3V
- R4 pad 1: Net-(J6-C) -> GND
- R4 pad 2: 3.3V -> Net-(J6-A)
Routing:
- net INT2: track 13.7 -> 16.8 mm, vias 2 -> 0
- net GND: track 2.44 -> 5.32 mm, vias 14 -> 15
- net Net-(J6-C): track 2.16 -> 0.00 mm, vias 1 -> 0
- net Net-(J6-A): track 0.00 -> 1.98 mm, vias 0 -> 1
- net ASDA: track 15.0 -> 15.3 mm, vias 2 -> 0
- net INT1: track 14.9 -> 15.1 mm, vias 2 -> 0
- net 3.3V: track 53.2 -> 53.1 mm, vias 4 -> 6
Other:
- board text added: "Finish: HASL Lead-Free"
- board text added: "Layers: 2"
- board text added: "Material: TG135"
- board text added: "Ordering Notes"
- board text added: "Outer Copper Weight: 1oz"
- board text added: "Released under the Creative Commons Attribution Share-Alike 4.0 License"
- board text added: "Silkscreen Color: White"
- board text added: "Solder Mask: Red"
- board text added: "Thickness: 1.6mm"
- board text added: "https://creativecommons.org/licenses/by-sa/4.0/"
