File: Hardware/Qwiic_BMA456.kicad_sch (KiCad schematic)
At the start: 27 parts, among them J0 LED, J1 Conn_01x04, J2 Qwiic_RA, J3 I²C, J4 Qwiic_RA, J5 Conn_01x06, J6 ADDR, U1 KX134

Commit message: Design Review Changes
Parts:
- U1: value KX134 -> BMA456; symbol Qwiic_KX13X-eagle-import:KX13X-KX134 -> SparkFun-Sensor:BMA456; PROD_ID IC-15486 -> IC-29229
Connections:
- net 3.3V: now also J6.3 (C); no longer R4.2
- net GND: now also R4.1; no longer J6.1 (A)
- new net: J6.1 (A), R4.2
Other:
- note added: "To enable SPI, cut both I²C and ADDR"
- moved on the sheet: R4
